File: SLI Bridge/KiCAD/SLI Interconnect PCB.kicad_pcb (KiCad board)
At the start: 2 copper layers, 52.9 x 43 mm, 4 parts, among them P1 Quantum3D SLI Port 1, P2 Reference SLI Male, P3 Quantum3D SLI Port 2, P4 Quantum3D SLI Port 3

Commit message: Update KiCAD Files
Routing:
- net /P7: track 52.1 -> 53.9 mm
- net /VD_184: vias 3 -> 1
- net GND: vias 49 -> 50
- net /VD_VSync: vias 2 -> 0
- net /VD_HSync: vias 3 -> 1
Other:
- board size 52.9 x 43 mm -> 52.9 x 45.1 mm
