File: SLI Bridge/KiCAD/SLI Interconnect PCB.kicad_sch (KiCad schematic)
At the start: 4 parts, among them P1 Quantum3D SLI Port 1, P2 Reference SLI Male, P3 Quantum3D SLI Port 2, P4 Quantum3D SLI Port 3

Commit message: Update KiCAD Files
Other:
- company: (none) -> Jeff Chen
- title: (none) -> Quantum3D Obsidian2 Adaptive SLI Bridge
Changed lines of the file:
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@@
 	(generator_version "8.0")
 	(paper "A4")
+	(title_block
+		(title "Quantum3D Obsidian2 Adaptive SLI Bridge")
+		(date "2024-11-07")
+		(rev "1.0")
+		(company "Jeff Chen")
+	)
 	(bus_alias "SLI"
 		(members "VD_185" "VD_186" "VD_HSync" "VD_VSync" "VD_184" "VD_201" "VD_214"
