File: VGA Input/KiCAD/VGA Input Board.kicad_sch (KiCad schematic)
At the start: 2 parts, among them P1 VGA_Male, P2 Quantum3D VGA Input

Commit message: Update KiCAD Files
Other:
- company: (none) -> Jeff Chen
- title: (none) -> Quantum3D Obsidian2 VGA Input PCB
Changed lines of the file:
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@@
 	(generator_version "8.0")
 	(paper "A4")
+	(title_block
+		(title "Quantum3D Obsidian2 VGA Input PCB")
+		(date "2024-11-07")
+		(rev "1.0")
+		(company "Jeff Chen")
+	)
 	(junction
 		(at 118.11 88.9)
