File: Xilinx CPLD Replacement/KiCAD/CPLD Replacement.kicad_sch (KiCad schematic)
At the start: 6 parts, among them U1 CD74HC4053PWR

Commit message: Update KiCAD Files
Other:
- company: (none) -> Jeff Chen
- title: (none) -> Quantum3D Obsidian2 Xlinx CPLD Replacement
Changed lines of the file:
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@@
 	(generator_version "8.0")
 	(paper "A4")
+	(title_block
+		(title "Quantum3D Obsidian2 Xlinx CPLD Replacement")
+		(date "2024-11-07")
+		(rev "1.0")
+		(company "Jeff Chen")
+	)
 	(junction
 		(at 147.32 139.7)
